File: FTL/parse/test.kicad_pcb (KiCad board)
At the start: 2 copper layers, 215.4 x 152.5 mm, 6 parts

Commit message: New testing file
Parts:
- renumbered C1 to C2
Changed lines of the file:
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@@
     (property "Sheetname" "")
     (attr through_hole)
-    (fp_text reference "C1" (at 12.5 -5.12) (layer "F.SilkS")
+    (fp_text reference "C2" (at 12.5 -5.12) (layer "F.SilkS")
         (effects (font (size 1 1) (thickness 0.15)))
     )
